File: reverse-pcb/hucard_pcb_v6.kicad_pcb (KiCad board)
At the start: 2 copper layers, 2 parts, among them J1 Conn_01x38_Pin, U1 SST39SF040-70-4C-WHE

Commit message: Iterating on reverse PCB
Parts:
- moved J1 1.50 mm to (47.0, 101.5)
Routing:
- net /GND: track 64.1 -> 27.3 mm, vias 2 -> 6
- net /VCC: track 132.2 -> 135.9 mm
- net /A0: track 66.9 -> 70.2 mm
- net /A7: track 53.7 -> 57.0 mm
- net /A15: track 60.3 -> 63.6 mm
- net /A6: track 52.6 -> 55.9 mm
- net unconnected-(J1-Pin_36-Pad36): track 72.3 -> 75.6 mm
- net /A16: track 61.5 -> 64.8 mm
- net /WE: track 94.4 -> 97.7 mm
- net /DQ7: track 74.2 -> 77.5 mm
- net /DQ6: track 70.4 -> 73.7 mm
- net /DQ5: track 67.6 -> 70.9 mm
- net /DQ4: track 65.1 -> 68.4 mm
- net /A9: track 90.2 -> 93.5 mm
- net /A3: track 65.9 -> 69.2 mm
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- added copper zone on B.Cu, net /GND
- added copper zone on F.Cu, net /GND
Other:
- board outline added: 54.1 x 85.4 mm
